File: picokey.kicad_sch (KiCad schematic)
At the start: 27 parts, among them P1 USB_C_Plug_USB2.0, U1 RP2350A, U10 WE-TVS-82400102, U14 TPS76933, Y1 12MHz SMD3225-4P

Commit message: First layout
Parts:
- added C10: 100n, Capacitor_SMD:C_0603_1608Metric, symbol Device:C_Small
- added D1: WS2812B, LED_SMD:LED_WS2812B-2020_PLCC4_2.0x2.0mm, symbol LED:WS2812B
- added R4: 1k, Resistor_SMD:R_0603_1608Metric, symbol Device:R_Small
- added SW1: Function, Button_Switch_SMD:SW_Push_SPST_NO_Alps_SKRK, symbol Switch:SW_Push
- L1: footprint (none) -> rt_Inductor:L_0806
- P1: footprint (none) -> rt_Connector_USB:USB_C_Plug_XKB_U261-121N-4BS2S
- U1: value RP2350A -> RP2354A
Connections:
- net +5V: now also C10.1, D1.1 (VDD)
- net GND: now also C10.2, D1.3 (VSS), SW1.1
- net XTAL: now reaches C30.1, R32.1, Y1.3
- net USB_DP_ESD: now reaches R2.1, U10.4
- net USB_DP_RP: now reaches R2.2, U1.52 (USB_DP)
- net VREG_LX: now reaches L1.2, U1.48 (VREG_LX)
- net SWDIO: now reaches TP2.1, U1.25 (SWDIO)
- net XIN: now reaches C29.1, U1.21 (XIN), Y1.1
- net XOUT: now reaches R32.2, U1.22 (XOUT)
- net SWCLK: now reaches TP1.1, U1.24 (SWCLK)
- net LED_DAT: now reaches U1.5 (GPIO3)
- net LED_DAT: now also D1.4 (DIN)
- net USB_DM_RP: now reaches R1.2, U1.51 (USB_DM)
- net BUTTON: now reaches U1.60 (QSPI_SS)
- net BUTTON: now also R4.2
- net USB_DM_ESD: now reaches R1.1, U10.6
- net USB_DP: now reaches P1.A6 (D+), U10.3
- net USB_DM: now reaches P1.A7 (D-), U10.1
- new net: R4.1, SW1.2
- no-connect marks 8 -> 38
Other:
- moved on the sheet: L1, P1
